File: KiCad/Linky_Tempo_HomeKit.kicad_pcb (KiCad board)
At the start: 2 copper layers, 111.8 x 78.7 mm, 22 parts, among them J1 TIC, J3 Main(1) + Fil pilote (3,5,7), J4 +3.3V, J5 GND, J6 SCL, J7 SDA, Q2 PN2222A, Q3 2N7000, SW1 Setup, SW2 Annul_Délestage, U2 LTV-814, U3 MOC3041M

Commit message: correction de bugs
Parts:
- R4: value 120Ω -> 220Ω; footprint Resistor_THT:R_Axial_DIN0207_L6.3mm_D2.5mm_P5.08mm_Vertical -> Resistor_THT:R_Axial_DIN0207_L6.3mm_D2.5mm_P10.16mm_Horizontal
- moved R4 6.35 mm to (152.4, 53.3), turned to 0 degrees
Connections:
- R4 pad 1: +3.3V -> Net-(U1-VIN)
Routing:
- net Net-(U1-VIN): track 61.0 -> 141.0 mm, vias 2 -> 4
- net +3.3V: track 88.9 -> 81.3 mm
- net Net-(R4-Pad2): track 15.2 -> 8.89 mm
