File: KiCad/Linky_Tempo_HomeKit.kicad_sch (KiCad schematic)
At the start: 22 parts, among them J1 TIC, J3 Main(1) + Fil pilote (3,5,7), J4 +3.3V, J5 GND, J6 SCL, J7 SDA, Q2 PN2222A, Q3 2N7000, SW1 Setup, SW2 Annul_Délestage, U2 LTV-814, U3 MOC3041M

Commit message: correction de bugs
Parts:
- R4: value 120Ω -> 220Ω; footprint Resistor_THT:R_Axial_DIN0207_L6.3mm_D2.5mm_P5.08mm_Vertical -> Resistor_THT:R_Axial_DIN0207_L6.3mm_D2.5mm_P10.16mm_Horizontal
Connections:
- net +3.3V: no longer R4.1
- net at R3.1, U1.1 (VIN), U2.4: now also R4.1
Changed lines of the file:
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@@
 		(color 0 0 0 0)
 	)
+	(junction
+		(at 147.32 36.83)
+		(diameter 0)
+		(color 0 0 0 0)
+	)
 	(no_connect
 		(at 109.22 86.36)
@@
 	(wire
 		(pts
-			(xy 95.25 55.88) (xy 109.22 55.88)
+			(xy 147.32 36.83) (xy 205.74 36.83)
 		)
 		(stroke
@@
 	(wire
 		(pts
-			(xy 25.4 41.91) (xy 43.18 41.91)
+			(xy 95.25 55.88) (xy 109.22 55.88)
 		)
 		(stroke
@@
 	(wire
 		(pts
-			(xy 198.12 128.27) (xy 187.96 128.27)
+			(xy 25.4 41.91) (xy 43.18 41.91)
 		)
 		(stroke
@@
 	(wire
 		(pts
-			(xy 153.67 68.58) (xy 153.67 121.92)
+			(xy 198.12 128.27) (xy 187.96 128.27)
 		)
 		(stroke
@@
 	(wire
 		(pts
-			(xy 97.79 133.35) (xy 97.79 139.7)
+			(xy 153.67 68.58) (xy 153.67 121.92)
 		)
 		(stroke
@@
 	(wire
 		(pts
-			(xy 143.51 130.81) (xy 143.51 139.7)
+			(xy 97.79 133.35) (xy 97.79 139.7)
 		)
 		(stroke
@@
 	(wire
 		(pts
-			(xy 60.96 41.91) (xy 60.96 77.47)
+			(xy 143.51 130.81) (xy 143.51 139.7)
 		)
 		(stroke
@@
 	(wire
 		(pts
-			(xy 165.1 58.42) (xy 165.1 74.93)
+			(xy 60.96 41.91) (xy 60.96 77.47)
 		)
 		(stroke
@@
 	(wire
 		(pts
-			(xy 135.89 58.42) (xy 165.1 58.42)
-		)
-		(stroke
-			(width 0)
-			(type default)
-		)
-	)
-	(wire
-		(pts
-			(xy 143.51 55.88) (xy 143.51 36.83)
+			(xy 135.89 58.42) (xy 147.32 58.42)
 		)
 		(stroke
@@
 	(wire
 		(pts
-			(xy 135.89 55.88) (xy 143.51 55.88)
+			(xy 135.89 55.88) (xy 147.32 55.88)
 		)
 		(stroke
@@
 	(wire
 		(pts
+			(xy 147.32 58.42) (xy 147.32 59.69)
+		)
+		(stroke
+			(width 0)
+			(type default)
+		)
+	)
+	(wire
+		(pts
 			(xy 143.51 78.74) (xy 135.89 78.74)
 		)
@@
 	(wire
 		(pts
-			(xy 95.25 60.96) (xy 95.25 58.42)
+			(xy 95.25 59.69) (xy 95.25 58.42)
 		)
 		(stroke
@@
 	(wire
 		(pts
-			(xy 205.74 102.87) (xy 205.74 105.41)
+			(xy 147.32 36.83) (xy 147.32 55.88)
+		)
+		(stroke
+			(width 0)
+			(type default)
+		)
+	)
+	(wire
+		(pts
+			(xy 205.74 36.83) (xy 205.74 105.41)
 		)
 		(stroke
@@
 	(wire
 		(pts
-			(xy 95.25 52.07) (xy 95.25 55.88)
+			(xy 95.25 54.61) (xy 95.25 55.88)
 		)
 		(stroke
@@
 	(wire
 		(pts
-			(xy 143.51 36.83) (xy 80.01 36.83)
+			(xy 80.01 36.83) (xy 147.32 36.83)
 		)
 		(stroke
@@
 			)
 		)
-		(property "Value" "120Ω"
+		(property "Value" "220Ω"
 			(at 208.28 110.4899 0)
 			(effects
@@
 			)
 		)
-		(property "Footprint" "Resistor_THT:R_Axial_DIN0207_L6.3mm_D2.5mm_P5.08mm_Vertical"
+		(property "Footprint" "Resistor_THT:R_Axial_DIN0207_L6.3mm_D2.5mm_P10.16mm_Horizontal"
 			(at 203.962 109.22 90)
 			(effects
@@
 	(symbol
 		(lib_id "power:+3.3V")
-		(at 205.74 102.87 0)
-		(unit 1)
-		(exclude_from_sim no)
-		(in_bom yes)
-		(on_board yes)
-		(dnp no)
-		(property "Reference" "#PWR010"
-			(at 205.74 106.68 0)
-			(effects
-				(font
-					(size 1.27 1.27)
-				)
-				(hide yes)
-			)
-		)
-		(property "Value" "+3.3V"
-			(at 205.74 97.79 0)
-			(effects
-				(font
-					(size 1.27 1.27)
-				)
-			)
-		)
-		(property "Footprint" ""
-			(at 205.74 102.87 0)
-			(effects
-				(font
-					(size 1.27 1.27)
-				)
-				(hide yes)
-			)
-		)
-		(property "Datasheet" ""
-			(at 205.74 102.87 0)
-			(effects
-				(font
-					(size 1.27 1.27)
-				)
-				(hide yes)
-			)
-		)
-		(property "Description" "Power symbol creates a global label with name \"+3.3V\""
-			(at 205.74 102.87 0)
-			(effects
-				(font
-					(size 1.27 1.27)
-				)
-				(hide yes)
-			)
-		)
-		(pin "1"
-		)
-		(instances
-			(project "Linky_Tempo_HomeKit"
-				(path "/9588d092-783d-4d3f-a96b-fb17d909e9c7"
-					(reference "#PWR010")
-					(unit 1)
-				)
-			)
-		)
-	)
-	(symbol
-		(lib_id "power:+3.3V")
-		(at 95.25 52.07 0)
+		(at 95.25 54.61 0)
 		(unit 1)
 		(exclude_from_sim no)
@@
 		(dnp no)
 		(property "Reference" "#PWR01"
-			(at 95.25 55.88 0)
+			(at 95.25 58.42 0)
 			(effects
 				(font
@@
 		)
 		(property "Value" "+3.3V"
-			(at 95.25 46.99 0)
+			(at 95.25 49.53 0)
 			(effects
 				(font
@@
 		)
 		(property "Footprint" ""
-			(at 95.25 52.07 0)
+			(at 95.25 54.61 0)
 			(effects
 				(font
@@
 		)
 		(property "Datasheet" ""
-			(at 95.25 52.07 0)
+			(at 95.25 54.61 0)
 			(effects
 				(font
@@
 		)
 		(property "Description" "Power symbol creates a global label with name \"+3.3V\""
-			(at 95.25 52.07 0)
+			(at 95.25 54.61 0)
 			(effects
 				(font
@@
 	(symbol
 		(lib_id "power:GND")
-		(at 165.1 74.93 0)
+		(at 147.32 59.69 0)
 		(unit 1)
 		(exclude_from_sim no)
@@
 		(fields_autoplaced yes)
 		(property "Reference" "#PWR04"
-			(at 165.1 81.28 0)
+			(at 147.32 66.04 0)
 			(effects
 				(font
@@
 		)
 		(property "Value" "GND"
-			(at 165.1 80.01 0)
+			(at 147.32 64.77 0)
 			(effects
 				(font
@@
 		)
 		(property "Footprint" ""
-			(at 165.1 74.93 0)
+			(at 147.32 59.69 0)
 			(effects
 				(font
@@
 		)
 		(property "Datasheet" ""
-			(at 165.1 74.93 0)
+			(at 147.32 59.69 0)
 			(effects
 				(font
@@
 		)
 		(property "Description" "Power symbol creates a global label with name \"GND\" , ground"
-			(at 165.1 74.93 0)
+			(at 147.32 59.69 0)
 			(effects
 				(font
@@
 	(symbol
 		(lib_id "power:GND")
-		(at 95.25 60.96 0)
+		(at 95.25 59.69 0)
 		(unit 1)
 		(exclude_from_sim no)
@@
 		(fields_autoplaced yes)
 		(property "Reference" "#PWR05"
-			(at 95.25 67.31 0)
+			(at 95.25 66.04 0)
 			(effects
 				(font
@@
 		)
 		(property "Value" "GND"
-			(at 95.25 66.04 0)
+			(at 95.25 64.77 0)
 			(effects
 				(font
@@
 		)
 		(property "Footprint" ""
-			(at 95.25 60.96 0)
+			(at 95.25 59.69 0)
 			(effects
 				(font
@@
 		)
 		(property "Datasheet" ""
-			(at 95.25 60.96 0)
+			(at 95.25 59.69 0)
 			(effects
 				(font
@@
 		)
 		(property "Description" "Power symbol creates a global label with name \"GND\" , ground"
-			(at 95.25 60.96 0)
+			(at 95.25 59.69 0)
 			(effects
 				(font
